Commit message: ur_macro.xacro, ur10e.srdf, joint_limits.yaml

File: ur_description/urdf/inc/ur_macro.xacro (robot description, xacro)
@@ -206,15 +206,45 @@
       </xacro:cylinder_inertial>
     </link>
+    <link name="cylinder_link">
+      <inertial>
+        <origin xyz="0 0 0.15" rpy="0 0 0"/>
+        <mass value="1"/>
+        <inertia ixx="0.1" ixy="0" ixz="0" iyy="0.1" iyz="0" izz="0.1"/>
+      </inertial>
+      <visual>
+        <origin xyz="0 0 0.1" rpy="0 0 0"/>
+        <geometry>
+          <cylinder length="0.3" radius="0.1"/>
+        </geometry>
+      </visual>
+      <collision>
+        <origin xyz="0 0 0.15" rpy="0 0 0"/>
+        <geometry>
+          <cylinder length="0.3" radius="0.1"/>
+        </geometry>
+      </collision>
+    </link>
+    <joint name="${prefix}base_link-cylinder_joint" type="fixed">
+      <parent link="${prefix}base_link"/>
+      <child link="cylinder_link"/>
+      <origin xyz="0 0 0" rpy="0 0 ${pi}"/>
+    </joint>
+    <joint name="${prefix}cylinder-base_link_inertia-joint" type="fixed">
+      <origin xyz="0 0 0.3" ryp="0 0 0" />
+      <parent link="cylinder_link" />
+      <child link="${prefix}base_link_inertia" />
+    </joint>
     <!-- joints: main serial chain -->
+    <!--
     <joint name="${prefix}base_link-base_link_inertia" type="fixed">
       <parent link="${prefix}base_link" />
       <child link="${prefix}base_link_inertia" />
-      <!-- 'base_link' is REP-103 aligned (so X+ forward), while the internal
+       'base_link' is REP-103 aligned (so X+ forward), while the internal
            frames of the robot/controller have X+ pointing backwards.
            Use the joint between 'base_link' and 'base_link_inertia' (a dummy
            link/frame) to introduce the necessary rotation over Z (of pi rad).
-      -->
       <origin xyz="0 0 0" rpy="0 0 ${pi}" />
     </joint>
+    -->
     <joint name="${prefix}shoulder_pan_joint" type="revolute">
       <parent link="${prefix}base_link_inertia" />
@@ -290,14 +320,21 @@
     </joint>
     <!-- ROS-Industrial 'base' frame: base_link to UR 'Base' Coordinates transform -->
+    <!--
     <link name="${prefix}base"/>
     <joint name="${prefix}base_link-base_fixed_joint" type="fixed">
-      <!-- Note the rotation over Z of pi radians: as base_link is REP-103
+       Note the rotation over Z of pi radians: as base_link is REP-103
            aligned (ie: has X+ forward, Y+ left and Z+ up), this is needed
            to correctly align 'base' with the 'Base' coordinate system of
            the UR controller.
-      -->
       <origin xyz="0 0 0" rpy="0 0 ${pi}"/>
       <parent link="${prefix}base_link"/>
       <child link="${prefix}base"/>
+    </joint>
+    -->
+    <link name="${prefix}base"/>
+    <joint name="${prefix}cylinder_link-base_joint" type="fixed">
+      <origin xyz="0 0 0.3" ryp="0 0 0" />
+      <parent link="cylinder_link" />
+      <child link="${prefix}base" />
     </joint>
     <!-- ROS-Industrial 'flange' frame: attachment point for EEF models -->
@@ -308,11 +345,21 @@
       <origin xyz="0 0 0" rpy="0 ${-pi/2.0} ${-pi/2.0}" />
     </joint>
-    <!-- ROS-Industrial 'tool0' frame: all-zeros tool frame -->
+    <!-- ROS-Industrial 'tool0' frame: all-zeros tool frame
     <link name="${prefix}tool0"/>
     <joint name="${prefix}flange-tool0" type="fixed">
-      <!-- default toolframe: X+ left, Y+ up, Z+ front -->
+      < default toolframe: X+ left, Y+ up, Z+ front
       <origin xyz="0 0 0" rpy="${pi/2.0} 0 ${pi/2.0}"/>
       <parent link="${prefix}flange"/>
       <child link="${prefix}tool0"/>
+    </joint>-->
+    <xacro:include filename="$(find ur10e_controller)/urdf/_d435.urdf.xacro" />
+    <xacro:sensor_d435 parent="${prefix}flange">
+      <origin xyz="-0.2 -0.1 0" rpy="${-pi/2} 0 ${-pi/4}"/>
+    </xacro:sensor_d435>
+    <link name="printer_link" />
+    <joint name="${prefix}flange-printer_link_joint" type="fixed">
+      <origin xyz="0.05 -0.15 0" rpy="${-pi/2} 0 0" />
+      <parent link="${prefix}flange" />
+      <child link="printer_link" />
     </joint>
   </xacro:macro>

Commit message: migrate

File: ur_description/urdf/inc/ur_macro.xacro (robot description, xacro)
@@ -228,5 +228,5 @@
       <parent link="${prefix}base_link"/>
       <child link="cylinder_link"/>
-      <origin xyz="0 0 0" rpy="0 0 ${pi}"/>
+      <origin xyz="0 0 0.15" rpy="0 0 ${pi}"/>
     </joint>
     <joint name="${prefix}cylinder-base_link_inertia-joint" type="fixed">

Commit message: wired connection

File: ur_description/urdf/inc/ur_macro.xacro (robot description, xacro)
@@ -228,5 +228,5 @@
       <parent link="${prefix}base_link"/>
       <child link="cylinder_link"/>
-      <origin xyz="0 0 0.15" rpy="0 0 ${pi}"/>
+      <origin xyz="0 0 0" rpy="0 0 ${pi}"/>
     </joint>
     <joint name="${prefix}cylinder-base_link_inertia-joint" type="fixed">

Commit message: hand-eye calibration

File: ur_description/urdf/inc/ur_macro.xacro (robot description, xacro)
@@ -64,5 +64,18 @@
     <xacro:ur_arm_transmission prefix="${prefix}" hw_interface="${transmission_hw_interface}" />
     <!-- links: main serial chain -->
-    <link name="${prefix}base_link"/>
+    <link name="${prefix}base_link">
+      <visual>
+        <origin xyz="0 0 0.15" rpy="0 0 0"/>
+        <geometry>
+          <cylinder length="0.3" radius="0.1"/>
+        </geometry>
+      </visual>
+      <collision>
+        <origin xyz="0 0 0.15" rpy="0 0 0"/>
+        <geometry>
+          <cylinder length="0.3" radius="0.1"/>
+        </geometry>
+      </collision>
+    </link>
     <link name="${prefix}base_link_inertia">
       <visual>
@@ -206,4 +219,5 @@
       </xacro:cylinder_inertial>
     </link>
+<!--
     <link name="cylinder_link">
       <inertial>
@@ -213,5 +227,5 @@
       </inertial>
       <visual>
-        <origin xyz="0 0 0.1" rpy="0 0 0"/>
+        <origin xyz="0 0 0.15" rpy="0 0 0"/>
         <geometry>
           <cylinder length="0.3" radius="0.1"/>
@@ -224,6 +238,6 @@
         </geometry>
       </collision>
-    </link>
-    <joint name="${prefix}base_link-cylinder_joint" type="fixed">
+    </link> -->
+    <!-- <joint name="${prefix}base_link-cylinder_joint" type="fixed">
       <parent link="${prefix}base_link"/>
       <child link="cylinder_link"/>
@@ -234,17 +248,16 @@
       <parent link="cylinder_link" />
       <child link="${prefix}base_link_inertia" />
-    </joint>
+    </joint> -->
     <!-- joints: main serial chain -->
-    <!--
     <joint name="${prefix}base_link-base_link_inertia" type="fixed">
       <parent link="${prefix}base_link" />
       <child link="${prefix}base_link_inertia" />
-       'base_link' is REP-103 aligned (so X+ forward), while the internal
+       <!-- 'base_link' is REP-103 aligned (so X+ forward), while the internal
            frames of the robot/controller have X+ pointing backwards.
            Use the joint between 'base_link' and 'base_link_inertia' (a dummy
            link/frame) to introduce the necessary rotation over Z (of pi rad).
-      <origin xyz="0 0 0" rpy="0 0 ${pi}" />
-    </joint>
-    -->
+       -->
+      <origin xyz="0 0 0.3" rpy="0 0 ${pi}" />
+    </joint>
     <joint name="${prefix}shoulder_pan_joint" type="revolute">
       <parent link="${prefix}base_link_inertia" />
@@ -320,22 +333,21 @@
     </joint>
     <!-- ROS-Industrial 'base' frame: base_link to UR 'Base' Coordinates transform -->
-    <!--
     <link name="${prefix}base"/>
     <joint name="${prefix}base_link-base_fixed_joint" type="fixed">
-       Note the rotation over Z of pi radians: as base_link is REP-103
+       <!-- Note the rotation over Z of pi radians: as base_link is REP-103
            aligned (ie: has X+ forward, Y+ left and Z+ up), this is needed
            to correctly align 'base' with the 'Base' coordinate system of
            the UR controller.
+       -->
       <origin xyz="0 0 0" rpy="0 0 ${pi}"/>
       <parent link="${prefix}base_link"/>
       <child link="${prefix}base"/>
     </joint>
-    -->
-    <link name="${prefix}base"/>
+    <!-- <link name="${prefix}base"/>
     <joint name="${prefix}cylinder_link-base_joint" type="fixed">
-      <origin xyz="0 0 0.3" ryp="0 0 0" />
+      <origin xyz="0 0 0.3" ryp="0 0 ${pi}" />
       <parent link="cylinder_link" />
       <child link="${prefix}base" />
-    </joint>
+    </joint> -->
     <!-- ROS-Industrial 'flange' frame: attachment point for EEF models -->
     <link name="${prefix}flange" />
@@ -355,9 +367,9 @@
     <xacro:include filename="$(find ur10e_controller)/urdf/_d435.urdf.xacro" />
     <xacro:sensor_d435 parent="${prefix}flange">
-      <origin xyz="-0.2 -0.1 0" rpy="${-pi/2} 0 ${-pi/4}"/>
+      <origin xyz="-0.12 -0.06 0.02" rpy="${-pi/2} 0 ${-pi/6}"/>
     </xacro:sensor_d435>
     <link name="printer_link" />
     <joint name="${prefix}flange-printer_link_joint" type="fixed">
-      <origin xyz="0.05 -0.15 0" rpy="${-pi/2} 0 0" />
+      <origin xyz="0 -0.15 0" rpy="${-pi/2} 0 0" />
       <parent link="${prefix}flange" />
       <child link="printer_link" />

Commit message: calibration

File: ur_description/urdf/inc/ur_macro.xacro (robot description, xacro)
@@ -365,8 +365,8 @@
       <child link="${prefix}tool0"/>
     </joint>-->
-    <xacro:include filename="$(find ur10e_controller)/urdf/_d435.urdf.xacro" />
+    <!-- <xacro:include filename="$(find ur10e_controller)/urdf/_d435.urdf.xacro" />
     <xacro:sensor_d435 parent="${prefix}flange">
-      <origin xyz="-0.12 -0.06 0.02" rpy="${-pi/2} 0 ${-pi/6}"/>
-    </xacro:sensor_d435>
+      <origin xyz="-0.06 -0.08 0.016" rpy="${-pi/2} 0 ${-pi/24}"/>
+    </xacro:sensor_d435>  -->
     <link name="printer_link" />
     <joint name="${prefix}flange-printer_link_joint" type="fixed">

Commit message: charuco calibration same error

File: ur_description/urdf/inc/ur_macro.xacro (robot description, xacro)
@@ -357,19 +357,19 @@
       <origin xyz="0 0 0" rpy="0 ${-pi/2.0} ${-pi/2.0}" />
     </joint>
-    <!-- ROS-Industrial 'tool0' frame: all-zeros tool frame
+    <!-- ROS-Industrial 'tool0' frame: all-zeros tool frame  -->
     <link name="${prefix}tool0"/>
     <joint name="${prefix}flange-tool0" type="fixed">
-      < default toolframe: X+ left, Y+ up, Z+ front
+      <!-- < default toolframe: X+ left, Y+ up, Z+ front  -->
       <origin xyz="0 0 0" rpy="${pi/2.0} 0 ${pi/2.0}"/>
       <parent link="${prefix}flange"/>
       <child link="${prefix}tool0"/>
-    </joint>-->
-    <!-- <xacro:include filename="$(find ur10e_controller)/urdf/_d435.urdf.xacro" />
+    </joint>
+    <xacro:include filename="$(find ur10e_controller)/urdf/_d435.urdf.xacro" />
     <xacro:sensor_d435 parent="${prefix}flange">
-      <origin xyz="-0.06 -0.08 0.016" rpy="${-pi/2} 0 ${-pi/24}"/>
-    </xacro:sensor_d435>  -->
+      <origin xyz="-0.06 -0.08 0.016" rpy="${-pi/2} 0 ${-pi/6}"/>
+    </xacro:sensor_d435>
     <link name="printer_link" />
     <joint name="${prefix}flange-printer_link_joint" type="fixed">
-      <origin xyz="0 -0.15 0" rpy="${-pi/2} 0 0" />
+      <origin xyz="0.05 -0.15 0" rpy="${-pi/2} 0 0" />
       <parent link="${prefix}flange" />
       <child link="printer_link" />

Commit message: parameter adjustment

File: ur_description/urdf/inc/ur_macro.xacro (robot description, xacro)
@@ -64,18 +64,5 @@
     <xacro:ur_arm_transmission prefix="${prefix}" hw_interface="${transmission_hw_interface}" />
     <!-- links: main serial chain -->
-    <link name="${prefix}base_link">
-      <visual>
-        <origin xyz="0 0 0.15" rpy="0 0 0"/>
-        <geometry>
-          <cylinder length="0.3" radius="0.1"/>
-        </geometry>
-      </visual>
-      <collision>
-        <origin xyz="0 0 0.15" rpy="0 0 0"/>
-        <geometry>
-          <cylinder length="0.3" radius="0.1"/>
-        </geometry>
-      </collision>
-    </link>
+    <link name="${prefix}base_link"/>
     <link name="${prefix}base_link_inertia">
       <visual>
@@ -219,44 +206,14 @@
       </xacro:cylinder_inertial>
     </link>
-<!--
-    <link name="cylinder_link">
-      <inertial>
-        <origin xyz="0 0 0.15" rpy="0 0 0"/>
-        <mass value="1"/>
-        <inertia ixx="0.1" ixy="0" ixz="0" iyy="0.1" iyz="0" izz="0.1"/>
-      </inertial>
-      <visual>
-        <origin xyz="0 0 0.15" rpy="0 0 0"/>
-        <geometry>
-          <cylinder length="0.3" radius="0.1"/>
-        </geometry>
-      </visual>
-      <collision>
-        <origin xyz="0 0 0.15" rpy="0 0 0"/>
-        <geometry>
-          <cylinder length="0.3" radius="0.1"/>
-        </geometry>
-      </collision>
-    </link> -->
-    <!-- <joint name="${prefix}base_link-cylinder_joint" type="fixed">
-      <parent link="${prefix}base_link"/>
-      <child link="cylinder_link"/>
-      <origin xyz="0 0 0" rpy="0 0 ${pi}"/>
-    </joint>
-    <joint name="${prefix}cylinder-base_link_inertia-joint" type="fixed">
-      <origin xyz="0 0 0.3" ryp="0 0 0" />
-      <parent link="cylinder_link" />
-      <child link="${prefix}base_link_inertia" />
-    </joint> -->
     <!-- joints: main serial chain -->
     <joint name="${prefix}base_link-base_link_inertia" type="fixed">
       <parent link="${prefix}base_link" />
       <child link="${prefix}base_link_inertia" />
-       <!-- 'base_link' is REP-103 aligned (so X+ forward), while the internal
+      <!-- 'base_link' is REP-103 aligned (so X+ forward), while the internal
            frames of the robot/controller have X+ pointing backwards.
            Use the joint between 'base_link' and 'base_link_inertia' (a dummy
            link/frame) to introduce the necessary rotation over Z (of pi rad).
-       -->
-      <origin xyz="0 0 0.3" rpy="0 0 ${pi}" />
+      -->
+      <origin xyz="0 0 0" rpy="0 0 ${pi}" />
     </joint>
     <joint name="${prefix}shoulder_pan_joint" type="revolute">
@@ -335,19 +292,13 @@
     <link name="${prefix}base"/>
     <joint name="${prefix}base_link-base_fixed_joint" type="fixed">
-       <!-- Note the rotation over Z of pi radians: as base_link is REP-103
+      <!-- Note the rotation over Z of pi radians: as base_link is REP-103
            aligned (ie: has X+ forward, Y+ left and Z+ up), this is needed
            to correctly align 'base' with the 'Base' coordinate system of
            the UR controller.
-       -->
+      -->
       <origin xyz="0 0 0" rpy="0 0 ${pi}"/>
       <parent link="${prefix}base_link"/>
       <child link="${prefix}base"/>
     </joint>
-    <!-- <link name="${prefix}base"/>
-    <joint name="${prefix}cylinder_link-base_joint" type="fixed">
-      <origin xyz="0 0 0.3" ryp="0 0 ${pi}" />
-      <parent link="cylinder_link" />
-      <child link="${prefix}base" />
-    </joint> -->
     <!-- ROS-Industrial 'flange' frame: attachment point for EEF models -->
     <link name="${prefix}flange" />
@@ -357,19 +308,15 @@
       <origin xyz="0 0 0" rpy="0 ${-pi/2.0} ${-pi/2.0}" />
     </joint>
-    <!-- ROS-Industrial 'tool0' frame: all-zeros tool frame  -->
+    <!-- ROS-Industrial 'tool0' frame: all-zeros tool frame -->
     <link name="${prefix}tool0"/>
     <joint name="${prefix}flange-tool0" type="fixed">
-      <!-- < default toolframe: X+ left, Y+ up, Z+ front  -->
+      <!-- default toolframe: X+ left, Y+ up, Z+ front -->
       <origin xyz="0 0 0" rpy="${pi/2.0} 0 ${pi/2.0}"/>
       <parent link="${prefix}flange"/>
       <child link="${prefix}tool0"/>
     </joint>
-    <xacro:include filename="$(find ur10e_controller)/urdf/_d435.urdf.xacro" />
-    <xacro:sensor_d435 parent="${prefix}flange">
-      <origin xyz="-0.06 -0.08 0.016" rpy="${-pi/2} 0 ${-pi/6}"/>
-    </xacro:sensor_d435>
     <link name="printer_link" />
     <joint name="${prefix}flange-printer_link_joint" type="fixed">
-      <origin xyz="0.05 -0.15 0" rpy="${-pi/2} 0 0" />
+      <origin xyz="0.065 -0.175 0" rpy="${-pi/2} 0 0" />
       <parent link="${prefix}flange" />
       <child link="printer_link" />

Commit message: printhead accurate position

File: ur_description/urdf/inc/ur_macro.xacro (robot description, xacro)
@@ -318,5 +318,5 @@
     <link name="printer_link" />
     <joint name="${prefix}flange-printer_link_joint" type="fixed">
-      <origin xyz="0.065 -0.175 0" rpy="${-pi/2} 0 0" />
+      <origin xyz="0.047 -0.171 0.00375" rpy="${-pi/2} 0 0" />
       <parent link="${prefix}flange" />
       <child link="printer_link" />
